Commit message: relax navigation params

File: src/auracle_description/urdf/robot_core.xacro (robot description, xacro)
@@ -34,5 +34,7 @@
         <parent link="base_link"/>
         <child link="chassis"/>
-        <origin xyz="0 0 0"/>
+        <!-- base_link sits on the WHEEL AXLE (the rotation centre of a diff drive). It used to be the rear edge of the chassis,
+             0.15 m behind the axle, which made odometry, SLAM, AMCL and Nav2 footprint checks all assume the wrong pivot. -->
+        <origin xyz="${-chassis_length/2} 0 0"/>
     </joint>
     <link name="chassis">
@@ -64,5 +66,5 @@
         <parent link="base_link"/>
         <child link="left_rocker"/>
-        <origin xyz="${chassis_length/2} ${chassis_width/2+rocker_width/2} 0" rpy="0 0 ${pi/2}" />
+        <origin xyz="0 ${chassis_width/2+rocker_width/2} 0" rpy="0 0 ${pi/2}" />
     </joint>
     <link name="left_rocker">
@@ -269,5 +271,5 @@
         <parent link="base_link"/>
         <child link="right_rocker"/>
-        <origin xyz="${chassis_length/2} ${-chassis_width/2-rocker_width/2} 0" rpy="0 0 ${pi/2}" />
+        <origin xyz="0 ${-chassis_width/2-rocker_width/2} 0" rpy="0 0 ${pi/2}" />
     </joint>
     <link name="right_rocker">

Commit message: update firmware

File: src/auracle_description/urdf/robot_core.xacro (robot description, xacro)
@@ -11,5 +11,5 @@
     <xacro:property name="tilted_link" value="0.1"/>
     <xacro:property name="rocker_mass" value="0.5"/>
-    <xacro:property name="wheel_radius" value="0.0239"/>
+    <xacro:property name="wheel_radius" value="0.0375"/>  <!-- 75 mm spiked wheels (2026-10-25); was 0.0239 -->
     <xacro:property name="wheel_thickness" value="0.026"/>
     <xacro:property name="wheel_mass" value="0.05"/>
@@ -27,5 +27,5 @@
         <parent link="base_footprint"/>
         <child link="base_link"/>
-        <origin xyz="0 0 0.0946" rpy="0 0 0"/>
+        <origin xyz="0 0 0.1082" rpy="0 0 0"/>  <!-- was 0.0946; +0.0136 m for the bigger wheels (0.0375 - 0.0239) -->
     </joint>
     <link name="base_link">

File: src/auracle_description/urdf/ros2_control.xacro (robot description, xacro)
@@ -15,5 +15,5 @@
                      "Calibrate ticks per rev". -->
                 <param name="left_enc_counts_per_rev">985.0</param>  <!-- hand-counted 2026-10-23: 10 turns = 9847 -->
-                <param name="right_enc_counts_per_rev">942.0</param>  <!-- hand-counted 2026-10-23: 10 turns = 9416 -->
+                <param name="right_enc_counts_per_rev">990.0</param>  <!-- re-counted 2026-10-25 (A+B): 9880 / 10 turns -->
                 <!-- Flip to -1.0 if a side's odom runs backwards when driving forward. -->
                 <param name="left_direction_sign">1.0</param>
